File: m0116.kicad_sch (KiCad schematic)
At the start: 255 parts, among them J2 Conn_01x04_MountingPin, J3 Conn_01x04_MountingPin, Q1 Q_PMOS_GSD AO3401A, Q2 Q_NMOS_GSD 2N7002, Q3 Q_NMOS_GSD 2N7002, Q4 2N3904, SW1 SW_Push, U1 XC6206P332MR, U2 74AHCT1G125, U3 STM32F411RETx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

Commit message: quasi-aek split layout
Parts:
- added SW_LALT_5: mx-alps-nec, Alps_Only:ALPS-1U, symbol MX_Alps_Hybrid:mx-alps-nec
- renumbered LED3 to LED1, LED1 to LED3
Connections:
- net COL3: now also SW_LALT_5.1 (COL)
- net at D98.2 (A), SW_LALT_1.2 (ROW), SW_LALT_2.2 (ROW)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: now also SW_LALT_5.2 (ROW)
Other:
- note added: "1.25 post-2.5"
- moved on the sheet: D2, D98
Changed lines of the file:
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@@
   (junction (at 33.02 295.91) (diameter 1.016) (color 0 0 0 0)
   )
-  (junction (at 93.98 406.4) (diameter 0) (color 0 0 0 0)
-  )
   (junction (at 86.36 342.9) (diameter 0) (color 0 0 0 0)
   )
@@
   (junction (at 88.9 104.14) (diameter 0) (color 0 0 0 0)
   )
+  (junction (at 78.74 405.13) (diameter 0) (color 0 0 0 0)
+  )
   (junction (at 134.62 285.75) (diameter 1.016) (color 0 0 0 0)
   )
@@
   (junction (at 176.53 377.19) (diameter 0) (color 0 0 0 0)
   )
+  (junction (at 110.49 414.02) (diameter 0) (color 0 0 0 0)
+  )
   (junction (at 160.02 396.24) (diameter 0) (color 0 0 0 0)
   )
@@
   (junction (at 71.12 358.14) (diameter 0) (color 0 0 0 0)
   )
-  (junction (at 290.83 276.86) (diameter 1.016) (color 0 0 0 0)
+  (junction (at 93.98 414.02) (diameter 0) (color 0 0 0 0)
   )
-  (junction (at 110.49 402.59) (diameter 0) (color 0 0 0 0)
+  (junction (at 290.83 276.86) (diameter 1.016) (color 0 0 0 0)
   )
   (junction (at 78.74 295.91) (diameter 1.016) (color 0 0 0 0)
@@
   (junction (at 48.26 276.86) (diameter 1.016) (color 0 0 0 0)
   )
-  (junction (at 78.74 406.4) (diameter 0) (color 0 0 0 0)
+  (junction (at 78.74 414.02) (diameter 0) (color 0 0 0 0)
   )
   (junction (at 55.88 285.75) (diameter 1.016) (color 0 0 0 0)
@@
   (junction (at 167.64 323.85) (diameter 0) (color 0 0 0 0)
   )
+  (junction (at 86.36 386.08) (diameter 0) (color 0 0 0 0)
+  )
   (junction (at 88.9 118.11) (diameter 0) (color 0 0 0 0)
   )
@@
     (stroke (width 0) (type solid))
   )
-  (wire (pts (xy 105.41 406.4) (xy 105.41 402.59))
-    (stroke (width 0) (type default))
-  )
   (wire (pts (xy 125.73 397.51) (xy 129.54 397.51))
     (stroke (width 0) (type default))
@@
     (stroke (width 0) (type default))
   )
-  (wire (pts (xy 63.5 406.4) (xy 78.74 406.4))
+  (wire (pts (xy 63.5 414.02) (xy 78.74 414.02))
     (stroke (width 0) (type default))
   )
-  (wire (pts (xy 78.74 406.4) (xy 93.98 406.4))
+  (wire (pts (xy 78.74 414.02) (xy 93.98 414.02))
     (stroke (width 0) (type default))
   )
@@
     (stroke (width 0) (type default))
   )
+  (wire (pts (xy 81.28 405.13) (xy 78.74 405.13))
+    (stroke (width 0) (type default))
+  )
   (wire (pts (xy 160.02 402.59) (xy 176.53 402.59))
     (stroke (width 0) (type default))
@@
     (stroke (width 0) (type default))
   )
-  (wire (pts (xy 93.98 384.81) (xy 93.98 406.4))
+  (wire (pts (xy 93.98 412.75) (xy 93.98 414.02))
     (stroke (width 0) (type default))
   )
@@
     (stroke (width 0) (type solid))
   )
-  (wire (pts (xy 93.98 347.98) (xy 93.98 379.73))
+  (wire (pts (xy 93.98 347.98) (xy 93.98 407.67))
     (stroke (width 0) (type default))
   )
@@
     (stroke (width 0) (type solid))
   )
-  (wire (pts (xy 105.41 402.59) (xy 110.49 402.59))
-    (stroke (width 0) (type default))
-  )
   (wire (pts (xy 124.46 144.78) (xy 125.73 144.78))
     (stroke (width 0) (type default))
@@
     (stroke (width 0) (type default))
   )
+  (wire (pts (xy 78.74 405.13) (xy 78.74 407.67))
+    (stroke (width 0) (type default))
+  )
   (wire (pts (xy 184.15 356.87) (xy 184.15 372.11))
     (stroke (width 0) (type default))
   )
-  (wire (pts (xy 110.49 401.32) (xy 110.49 402.59))
+  (wire (pts (xy 110.49 401.32) (xy 110.49 414.02))
     (stroke (width 0) (type default))
   )
@@
     (stroke (width 0) (type default))
   )
-  (wire (pts (xy 110.49 431.8) (xy 110.49 402.59))
+  (wire (pts (xy 110.49 431.8) (xy 110.49 414.02))
     (stroke (width 0) (type default))
   )
@@
     (stroke (width 0) (type default))
   )
+  (wire (pts (xy 78.74 391.16) (xy 78.74 405.13))
+    (stroke (width 0) (type default))
+  )
   (wire (pts (xy 307.34 361.95) (xy 307.34 375.92))
     (stroke (width 0) (type default))
@@
     (stroke (width 0) (type default))
   )
+  (wire (pts (xy 86.36 386.08) (xy 86.36 400.05))
+    (stroke (width 0) (type default))
+  )
   (wire (pts (xy 209.55 290.83) (xy 212.09 290.83))
     (stroke (width 0) (type solid))
@@
     (stroke (width 0) (type default))
   )
-  (wire (pts (xy 78.74 391.16) (xy 78.74 397.51))
-    (stroke (width 0) (type default))
-  )
   (wire (pts (xy 265.43 323.85) (xy 265.43 342.9))
     (stroke (width 0) (type solid))
@@
     (stroke (width 0) (type default))
   )
-  (wire (pts (xy 63.5 406.4) (xy 63.5 388.62))
+  (wire (pts (xy 63.5 388.62) (xy 63.5 414.02))
     (stroke (width 0) (type default))
   )
@@
     (stroke (width 0) (type solid))
   )
+  (wire (pts (xy 93.98 414.02) (xy 110.49 414.02))
+    (stroke (width 0) (type default))
+  )
   (wire (pts (xy 124.46 132.08) (xy 125.73 132.08))
     (stroke (width 0) (type default))
@@
     (stroke (width 0) (type default))
   )
-  (wire (pts (xy 78.74 402.59) (xy 78.74 406.4))
+  (wire (pts (xy 78.74 412.75) (xy 78.74 414.02))
     (stroke (width 0) (type default))
   )
@@
     (stroke (width 0) (type solid))
   )
-  (wire (pts (xy 93.98 406.4) (xy 105.41 406.4))
-    (stroke (width 0) (type default))
-  )
   (wire (pts (xy 176.53 290.83) (xy 179.07 290.83))
     (stroke (width 0) (type solid))
@@
     (effects (font (size 1.27 1.27)) (justify left bottom))
   )
+  (text "1.25 post-2.5" (at 83.82 405.13 0)
+    (effects (font (size 1.27 1.27)) (justify left bottom))
+  )
   (label "3.3V" (at 254 200.66 180) (fields_autoplaced)
     (effects (font (size 1.27 1.27)) (justify right bottom))
@@
   (symbol (lib_id "ws2812b:WS2812B") (at 274.32 135.89 0) (unit 1)
     (in_bom yes) (on_board yes) (dnp no)
-    (property "Reference" "LED1" (at 274.32 123.5202 0)
+    (property "Reference" "LED3" (at 274.32 123.5202 0)
       (effects (font (size 1.524 1.524)))
     )
@@
       (project "m0116"
         (path "/151da08b-0979-4785-a9bf-6fa9b165d629"
-          (reference "LED1") (unit 1)
+          (reference "LED3") (unit 1)
         )
       )
@@
     )
   )
-  (symbol (lib_id "Device:D_Small") (at 93.98 382.27 90) (unit 1)
+  (symbol (lib_id "Device:D_Small") (at 93.98 410.21 90) (unit 1)
     (in_bom yes) (on_board yes) (dnp no)
-    (property "Reference" "D2" (at 95.758 381.1016 90)
+    (property "Reference" "D2" (at 95.758 409.0416 90)
       (effects (font (size 1.27 1.27)) (justify right))
     )
-    (property "Value" "D_Small" (at 95.758 383.413 90)
+    (property "Value" "D_Small" (at 95.758 411.353 90)
       (effects (font (size 1.27 1.27)) (justify right))
     )
-    (property "Footprint" "Diode_SMD:D_SOD-123" (at 93.98 382.27 90)
+    (property "Footprint" "Diode_SMD:D_SOD-123" (at 93.98 410.21 90)
       (effects (font (size 1.27 1.27)) hide)
     )
-    (property "Datasheet" "~" (at 93.98 382.27 90)
+    (property "Datasheet" "~" (at 93.98 410.21 90)
       (effects (font (size 1.27 1.27)) hide)
     )
@@
     )
   )
-  (symbol (lib_id "Device:D_Small") (at 78.74 400.05 90) (unit 1)
+  (symbol (lib_id "Device:D_Small") (at 78.74 410.21 90) (unit 1)
     (in_bom yes) (on_board yes) (dnp no)
-    (property "Reference" "D98" (at 80.518 398.8816 90)
+    (property "Reference" "D98" (at 80.518 409.0416 90)
       (effects (font (size 1.27 1.27)) (justify right))
     )
-    (property "Value" "D_Small" (at 80.518 401.193 90)
+    (property "Value" "D_Small" (at 80.518 411.353 90)
       (effects (font (size 1.27 1.27)) (justify right))
     )
-    (property "Footprint" "Diode_SMD:D_SOD-123" (at 78.74 400.05 90)
+    (property "Footprint" "Diode_SMD:D_SOD-123" (at 78.74 410.21 90)
       (effects (font (size 1.27 1.27)) hide)
     )
-    (property "Datasheet" "~" (at 78.74 400.05 90)
+    (property "Datasheet" "~" (at 78.74 410.21 90)
       (effects (font (size 1.27 1.27)) hide)
     )
@@
   (symbol (lib_id "ws2812b:WS2812B") (at 345.44 135.89 0) (unit 1)
     (in_bom yes) (on_board yes) (dnp no)
-    (property "Reference" "LED3" (at 345.44 123.5202 0)
+    (property "Reference" "LED1" (at 345.44 123.5202 0)
       (effects (font (size 1.524 1.524)))
     )
@@
       (project "m0116"
         (path "/151da08b-0979-4785-a9bf-6fa9b165d629"
-          (reference "LED3") (unit 1)
+          (reference "LED1") (unit 1)
         )
       )
@@
   (symbol (lib_id "power:GND") (at 287.02 147.32 0) (unit 1)
     (in_bom yes) (on_board yes) (dnp no)
-    (property "Reference" "#PWR0119" (at 287.02 153.67 0)
+    (property "Reference" "#PWR0128" (at 287.02 153.67 0)
       (effects (font (size 1.27 1.27)) hide)
     )
@@
       (project "m0116"
         (path "/151da08b-0979-4785-a9bf-6fa9b165d629"
-          (reference "#PWR0119") (unit 1)
+          (reference "#PWR0128") (unit 1)
         )
       )
@@
     )
   )
+  (symbol (lib_id "MX_Alps_Hybrid:mx-alps-nec") (at 82.55 401.32 0) (unit 1)
+    (in_bom yes) (on_board yes) (dnp no)
+    (property "Reference" "SW_LALT_5" (at 83.3882 395.6558 0)
+      (effects (font (size 1.524 1.524)))
+    )
+    (property "Value" "mx-alps-nec" (at 83.3882 397.5354 0)
+      (effects (font (size 0.508 0.508)))
+    )
+    (property "Footprint" "Alps_Only:ALPS-1U" (at 66.675 401.955 0)
+      (effects (font (size 1.524 1.524)) hide)
+    )
+    (property "Datasheet" "" (at 66.675 401.955 0)
+      (effects (font (size 1.524 1.524)) hide)
+    )
+    (pin "1")
+    (pin "2")
+    (instances
+      (project "m0116"
+        (path "/151da08b-0979-4785-a9bf-6fa9b165d629"
+          (reference "SW_LALT_5") (unit 1)
+        )
+      )
+    )
+  )
   (symbol (lib_id "power:GND") (at 237.49 118.11 90) (unit 1)
     (in_bom yes) (on_board yes) (dnp no)
-    (property "Reference" "#PWR0101" (at 243.84 118.11 0)
+    (property "Reference" "#PWR0127" (at 243.84 118.11 0)
       (effects (font (size 1.27 1.27)) hide)
     )
@@
       (project "m0116"
         (path "/151da08b-0979-4785-a9bf-6fa9b165d629"
-          (reference "#PWR0101") (unit 1)
+          (reference "#PWR0127") (unit 1)
         )
       )

Commit message: update
Other:
- note added: "1.5u for quasi aek 2"
- note added: "6.25u at101w for quasi aek 2"
- note removed: "1.5u"
- note removed: "6.25u at101w"
- moved on the sheet: D99
Changed lines of the file:
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@@
   (junction (at 257.81 361.95) (diameter 0) (color 0 0 0 0)
   )
-  (junction (at 125.73 431.8) (diameter 0) (color 0 0 0 0)
+  (junction (at 125.73 427.99) (diameter 0) (color 0 0 0 0)
   )
   (junction (at 127 328.93) (diameter 0) (color 0 0 0 0)
@@
     (stroke (width 0) (type default))
   )
+  (wire (pts (xy 110.49 401.32) (xy 110.49 414.02))
+    (stroke (width 0) (type default))
+  )
   (wire (pts (xy 88.9 104.14) (xy 107.95 104.14))
     (stroke (width 0) (type default))
@@
     (stroke (width 0) (type default))
   )
-  (wire (pts (xy 110.49 401.32) (xy 110.49 414.02))
-    (stroke (width 0) (type default))
-  )
   (wire (pts (xy 93.98 271.78) (xy 96.52 271.78))
     (stroke (width 0) (type solid))
@@
     (stroke (width 0) (type default))
   )
-  (wire (pts (xy 110.49 431.8) (xy 110.49 414.02))
+  (wire (pts (xy 110.49 427.99) (xy 110.49 414.02))
     (stroke (width 0) (type default))
   )
@@
     (stroke (width 0) (type default))
   )
-  (wire (pts (xy 143.51 431.8) (xy 143.51 402.59))
+  (wire (pts (xy 143.51 427.99) (xy 143.51 402.59))
     (stroke (width 0) (type default))
   )
@@
     (stroke (width 0) (type solid))
   )
-  (wire (pts (xy 110.49 431.8) (xy 125.73 431.8))
+  (wire (pts (xy 110.49 427.99) (xy 125.73 427.99))
     (stroke (width 0) (type default))
   )
@@
     (stroke (width 0) (type solid))
   )
-  (wire (pts (xy 125.73 431.8) (xy 143.51 431.8))
+  (wire (pts (xy 125.73 427.99) (xy 143.51 427.99))
     (stroke (width 0) (type default))
   )
@@
     (stroke (width 0) (type default))
   )
-  (wire (pts (xy 125.73 426.72) (xy 125.73 416.56))
+  (wire (pts (xy 125.73 422.91) (xy 125.73 416.56))
     (stroke (width 0) (type default))
   )
@@
     (effects (font (size 1.27 1.27)) (justify left bottom))
   )
-  (text "6.25u at101w" (at 133.35 378.46 0)
+  (text "6.25u at101w\nfor quasi aek 2" (at 133.35 379.73 0)
     (effects (font (size 1.27 1.27)) (justify left bottom))
   )
@@
     (effects (font (size 1.27 1.27)) (justify left bottom))
   )
-  (text "1.5u\n" (at 165.1 378.46 0)
+  (text "1.5u\nfor quasi aek 2\n" (at 162.56 381 0)
     (effects (font (size 1.27 1.27)) (justify left bottom))
   )
@@
     )
   )
-  (symbol (lib_id "Device:D_Small") (at 125.73 429.26 90) (unit 1)
+  (symbol (lib_id "Device:D_Small") (at 125.73 425.45 90) (unit 1)
     (in_bom yes) (on_board yes) (dnp no)
-    (property "Reference" "D99" (at 127.508 428.0916 90)
+    (property "Reference" "D99" (at 127.508 424.2816 90)
       (effects (font (size 1.27 1.27)) (justify right))
     )
-    (property "Value" "D_Small" (at 127.508 430.403 90)
+    (property "Value" "D_Small" (at 127.508 426.593 90)
       (effects (font (size 1.27 1.27)) (justify right))
     )
-    (property "Footprint" "Diode_SMD:D_SOD-123" (at 125.73 429.26 90)
+    (property "Footprint" "Diode_SMD:D_SOD-123" (at 125.73 425.45 90)
       (effects (font (size 1.27 1.27)) hide)
     )
-    (property "Datasheet" "~" (at 125.73 429.26 90)
+    (property "Datasheet" "~" (at 125.73 425.45 90)
       (effects (font (size 1.27 1.27)) hide)
     )
