File: m0116.kicad_sch (KiCad schematic)
At the start: 256 parts, among them J2 Conn_01x04_MountingPin, J3 Conn_01x04_MountingPin, Q1 Q_PMOS_GSD AO3401A, Q2 Q_NMOS_GSD 2N7002, Q3 Q_NMOS_GSD 2N7002, Q4 2N3904, SW1 SW_Push, U1 XC6206P332MR, U2 74AHCT1G125, U3 STM32F411RETx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

Commit message: fix
Parts:
- added SW_SP1_2, SW_SP2_6, SW_SP3_2: mx-alps-nec, Alps_Only:ALPS-1U, symbol MX_Alps_Hybrid:mx-alps-nec
Connections:
- net COL4: now also SW_SP1_2.1 (COL)
- net COL6: now also SW_SP2_6.1 (COL)
- net COL7: now also SW_SP3_2.1 (COL)
- net at D2.2 (A), SW_SP1_1.2 (ROW): now also SW_SP1_2.2 (ROW)
- net at D6.2 (A), SW_SP3_1.2 (ROW): now also SW_SP3_2.2 (ROW)
- net at D99.2 (A), SW_SP2_1.2 (ROW), SW_SP2_2.2 (ROW)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: now also SW_SP2_6.2 (ROW)
Other:
- note added: "split m0116 #2"
- moved on the sheet: D99
Changed lines of the file:
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@@
   (junction (at 160.02 377.19) (diameter 0) (color 0 0 0 0)
   )
+  (junction (at 93.98 363.22) (diameter 0) (color 0 0 0 0)
+  )
   (junction (at 204.47 65.405) (diameter 0) (color 0 0 0 0)
   )
@@
   (junction (at 86.36 342.9) (diameter 0) (color 0 0 0 0)
   )
+  (junction (at 151.13 342.9) (diameter 0) (color 0 0 0 0)
+  )
   (junction (at 118.11 266.7) (diameter 0) (color 0 0 0 0)
   )
@@
   (junction (at 257.81 361.95) (diameter 0) (color 0 0 0 0)
   )
-  (junction (at 125.73 427.99) (diameter 0) (color 0 0 0 0)
+  (junction (at 125.73 448.31) (diameter 0) (color 0 0 0 0)
   )
   (junction (at 127 328.93) (diameter 0) (color 0 0 0 0)
@@
   (junction (at 33.02 276.86) (diameter 1.016) (color 0 0 0 0)
   )
+  (junction (at 101.6 342.9) (diameter 0) (color 0 0 0 0)
+  )
   (junction (at 101.6 304.8) (diameter 0) (color 0 0 0 0)
   )
@@
   (junction (at 332.74 118.11) (diameter 0) (color 0 0 0 0)
   )
+  (junction (at 134.62 411.48) (diameter 0) (color 0 0 0 0)
+  )
   (junction (at 55.88 358.14) (diameter 0) (color 0 0 0 0)
   )
@@
   (junction (at 93.98 414.02) (diameter 0) (color 0 0 0 0)
   )
+  (junction (at 125.73 434.34) (diameter 0) (color 0 0 0 0)
+  )
   (junction (at 290.83 276.86) (diameter 1.016) (color 0 0 0 0)
   )
@@
   (junction (at 36.83 35.56) (diameter 0) (color 0 0 0 0)
   )
+  (junction (at 143.51 361.95) (diameter 0) (color 0 0 0 0)
+  )
   (junction (at 217.17 323.85) (diameter 0) (color 0 0 0 0)
   )
@@
     (stroke (width 0) (type solid))
   )
-  (wire (pts (xy 93.98 347.98) (xy 93.98 407.67))
+  (wire (pts (xy 93.98 347.98) (xy 93.98 363.22))
     (stroke (width 0) (type default))
   )
@@
     (stroke (width 0) (type solid))
   )
+  (wire (pts (xy 125.73 434.34) (xy 125.73 416.56))
+    (stroke (width 0) (type default))
+  )
   (wire (pts (xy 118.11 259.08) (xy 118.11 266.7))
     (stroke (width 0) (type default))
@@
     (stroke (width 0) (type default))
   )
-  (wire (pts (xy 110.49 427.99) (xy 110.49 414.02))
+  (wire (pts (xy 110.49 448.31) (xy 110.49 414.02))
     (stroke (width 0) (type default))
   )
@@
     (stroke (width 0) (type default))
   )
+  (wire (pts (xy 125.73 434.34) (xy 129.54 434.34))
+    (stroke (width 0) (type default))
+  )
   (wire (pts (xy 184.785 36.83) (xy 172.72 36.83))
     (stroke (width 0) (type default))
@@
     (stroke (width 0) (type solid))
   )
+  (wire (pts (xy 134.62 411.48) (xy 134.62 429.26))
+    (stroke (width 0) (type default))
+  )
   (wire (pts (xy 49.53 153.67) (xy 49.53 157.48))
     (stroke (width 0) (type default))
@@
     (stroke (width 0) (type solid))
   )
+  (wire (pts (xy 93.98 363.22) (xy 96.52 363.22))
+    (stroke (width 0) (type default))
+  )
   (wire (pts (xy 33.02 271.78) (xy 35.56 271.78))
     (stroke (width 0) (type solid))
@@
     (stroke (width 0) (type default))
   )
-  (wire (pts (xy 143.51 427.99) (xy 143.51 402.59))
+  (wire (pts (xy 143.51 448.31) (xy 143.51 402.59))
     (stroke (width 0) (type default))
   )
@@
     (stroke (width 0) (type default))
   )
+  (wire (pts (xy 143.51 361.95) (xy 143.51 397.51))
+    (stroke (width 0) (type default))
+  )
   (wire (pts (xy 176.53 328.93) (xy 179.07 328.93))
     (stroke (width 0) (type solid))
@@
     (stroke (width 0) (type default))
   )
-  (wire (pts (xy 143.51 347.98) (xy 143.51 397.51))
+  (wire (pts (xy 143.51 347.98) (xy 143.51 361.95))
     (stroke (width 0) (type default))
   )
@@
     (stroke (width 0) (type solid))
   )
-  (wire (pts (xy 110.49 427.99) (xy 125.73 427.99))
+  (wire (pts (xy 110.49 448.31) (xy 125.73 448.31))
     (stroke (width 0) (type default))
   )
@@
     (stroke (width 0) (type solid))
   )
-  (wire (pts (xy 125.73 427.99) (xy 143.51 427.99))
+  (wire (pts (xy 125.73 448.31) (xy 143.51 448.31))
     (stroke (width 0) (type default))
   )
@@
     (stroke (width 0) (type solid))
   )
+  (wire (pts (xy 93.98 363.22) (xy 93.98 407.67))
+    (stroke (width 0) (type default))
+  )
   (wire (pts (xy 85.09 84.455) (xy 87.63 84.455))
     (stroke (width 0) (type default))
@@
     (stroke (width 0) (type default))
   )
+  (wire (pts (xy 143.51 361.95) (xy 146.05 361.95))
+    (stroke (width 0) (type default))
+  )
   (wire (pts (xy 124.46 132.08) (xy 125.73 132.08))
     (stroke (width 0) (type default))
@@
     (stroke (width 0) (type solid))
   )
+  (wire (pts (xy 101.6 342.9) (xy 101.6 358.14))
+    (stroke (width 0) (type default))
+  )
   (wire (pts (xy 55.88 304.8) (xy 55.88 323.85))
     (stroke (width 0) (type solid))
@@
     (stroke (width 0) (type default))
   )
-  (wire (pts (xy 125.73 422.91) (xy 125.73 416.56))
+  (wire (pts (xy 125.73 443.23) (xy 125.73 434.34))
     (stroke (width 0) (type default))
   )
@@
     (stroke (width 0) (type default))
   )
+  (wire (pts (xy 151.13 342.9) (xy 151.13 356.87))
+    (stroke (width 0) (type default))
+  )
   (wire (pts (xy 226.06 381) (xy 242.57 381))
     (stroke (width 0) (type solid))
@@
     (effects (font (size 1.27 1.27)) (justify left bottom))
   )
+  (text "split m0116 #2\n" (at 146.05 363.22 0)
+    (effects (font (size 1.27 1.27)) (justify left bottom))
+  )
   (text "aek\n" (at 53.34 363.22 0)
     (effects (font (size 1.27 1.27)) (justify left bottom))
@@
     (effects (font (size 1.27 1.27)) (justify left bottom))
   )
+  (text "split m0116 #2" (at 100.33 363.22 0)
+    (effects (font (size 1.27 1.27)) (justify left bottom))
+  )
   (text "6.5u aek" (at 132.08 363.22 0)
     (effects (font (size 1.27 1.27)) (justify left bottom))
@@
     (effects (font (size 1.27 1.27)) (justify left bottom))
   )
+  (text "split m0116 #2" (at 134.62 434.34 0)
+    (effects (font (size 1.27 1.27)) (justify left bottom))
+  )
   (text "Has resistor in case this pin accidentally\ngets configured as output and gets pulled up"
     (at 52.07 182.88 0)
@@
     )
   )
-  (symbol (lib_id "Device:D_Small") (at 125.73 425.45 90) (unit 1)
+  (symbol (lib_id "Device:D_Small") (at 125.73 445.77 90) (unit 1)
     (in_bom yes) (on_board yes) (dnp no)
-    (property "Reference" "D99" (at 127.508 424.2816 90)
+    (property "Reference" "D99" (at 127.508 444.6016 90)
       (effects (font (size 1.27 1.27)) (justify right))
     )
-    (property "Value" "D_Small" (at 127.508 426.593 90)
+    (property "Value" "D_Small" (at 127.508 446.913 90)
       (effects (font (size 1.27 1.27)) (justify right))
     )
-    (property "Footprint" "Diode_SMD:D_SOD-123" (at 125.73 425.45 90)
+    (property "Footprint" "Diode_SMD:D_SOD-123" (at 125.73 445.77 90)
       (effects (font (size 1.27 1.27)) hide)
     )
-    (property "Datasheet" "~" (at 125.73 425.45 90)
+    (property "Datasheet" "~" (at 125.73 445.77 90)
       (effects (font (size 1.27 1.27)) hide)
     )
@@
     )
   )
+  (symbol (lib_id "MX_Alps_Hybrid:mx-alps-nec") (at 97.79 359.41 0) (unit 1)
+    (in_bom yes) (on_board yes) (dnp no)
+    (property "Reference" "SW_SP1_2" (at 98.6282 353.7458 0)
+      (effects (font (size 1.524 1.524)))
+    )
+    (property "Value" "mx-alps-nec" (at 98.6282 355.6254 0)
+      (effects (font (size 0.508 0.508)))
+    )
+    (property "Footprint" "Alps_Only:ALPS-1U" (at 81.915 360.045 0)
+      (effects (font (size 1.524 1.524)) hide)
+    )
+    (property "Datasheet" "" (at 81.915 360.045 0)
+      (effects (font (size 1.524 1.524)) hide)
+    )
+    (pin "1")
+    (pin "2")
+    (instances
+      (project "m0116"
+        (path "/151da08b-0979-4785-a9bf-6fa9b165d629"
+          (reference "SW_SP1_2") (unit 1)
+        )
+      )
+    )
+  )
   (symbol (lib_id "Device:C_Small") (at 228.6 118.11 270) (unit 1)
     (in_bom yes) (on_board yes) (dnp no)
@@
     )
   )
+  (symbol (lib_id "MX_Alps_Hybrid:mx-alps-nec") (at 130.81 430.53 0) (unit 1)
+    (in_bom yes) (on_board yes) (dnp no)
+    (property "Reference" "SW_SP2_6" (at 131.6482 424.8658 0)
+      (effects (font (size 1.524 1.524)))
+    )
+    (property "Value" "mx-alps-nec" (at 131.6482 426.7454 0)
+      (effects (font (size 0.508 0.508)))
+    )
+    (property "Footprint" "Alps_Only:ALPS-1U" (at 114.935 431.165 0)
+      (effects (font (size 1.524 1.524)) hide)
+    )
+    (property "Datasheet" "" (at 114.935 431.165 0)
+      (effects (font (size 1.524 1.524)) hide)
+    )
+    (pin "1")
+    (pin "2")
+    (instances
+      (project "m0116"
+        (path "/151da08b-0979-4785-a9bf-6fa9b165d629"
+          (reference "SW_SP2_6") (unit 1)
+        )
+      )
+    )
+  )
   (symbol (lib_id "MX_Alps_Hybrid:mx-alps-nec") (at 82.55 401.32 0) (unit 1)
     (in_bom yes) (on_board yes) (dnp no)
@@
         )
       )
+    )
+  )
+  (symbol (lib_id "MX_Alps_Hybrid:mx-alps-nec") (at 147.32 358.14 0) (unit 1)
+    (in_bom yes) (on_board yes) (dnp no)
+    (property "Reference" "SW_SP3_2" (at 148.1582 352.4758 0)
+      (effects (font (size 1.524 1.524)))
+    )
+    (property "Value" "mx-alps-nec" (at 148.1582 354.3554 0)
+      (effects (font (size 0.508 0.508)))
+    )
+    (property "Footprint" "Alps_Only:ALPS-1U" (at 131.445 358.775 0)
+      (effects (font (size 1.524 1.524)) hide)
+    )
+    (property "Datasheet" "" (at 131.445 358.775 0)
+      (effects (font (size 1.524 1.524)) hide)
+    )
+    (pin "1")
+    (pin "2")
+    (instances
+      (project "m0116"
+        (path "/151da08b-0979-4785-a9bf-6fa9b165d629"
+          (reference "SW_SP3_2") (unit 1)
+        )
+      )

Commit message: updates
Parts:
- added J1, J4: Conn_01x04, Connector_PinHeader_1.27mm:PinHeader_1x04_P1.27mm_Vertical, symbol Connector_Generic:Conn_01x04
- added J7: Conn_01x05, Connector_PinHeader_1.27mm:PinHeader_1x05_P1.27mm_Vertical, symbol Connector_Generic:Conn_01x05
Connections:
- net PA10: now also J1.4 (Pin_4)
- net PC2: now reaches U3.10 (PC2)
- net PC2: now also J7.1 (Pin_1)
- net PC3: now reaches U3.11 (PC3)
- net PC3: now also J7.4 (Pin_4)
- net PA1: now reaches U3.15 (PA1)
- net PA1: now also J7.3 (Pin_3)
- net PC13: now reaches U3.2 (PC13)
- net PC13: now also J4.4 (Pin_4)
- net PC4: now reaches U3.24 (PC4)
- net PC4: now also J7.5 (Pin_5)
- net PC14: now reaches U3.3 (PC14)
- net PC14: now also J4.3 (Pin_3)
- net PC15: now reaches U3.4 (PC15)
- net PC15: now also J4.1 (Pin_1)
- net PC12: now reaches U3.53 (PC12)
- net PC12: now also J1.1 (Pin_1)
- net PD2: now reaches U3.54 (PD2)
- net PD2: now also J1.2 (Pin_2)
- net PB6: now reaches U3.58 (PB6)
- net PB6: now also J1.3 (Pin_3)
- net PC0: now reaches U3.8 (PC0)
- net PC0: now also J7.2 (Pin_2)
- net PC1: now reaches U3.9 (PC1)
- net PC1: now also J4.2 (Pin_2)
- no-connect marks 16 -> 4
Other:
- note added: "Unused GPIO pins for extension"
- moved on the sheet: R17

Commit message: updates
Parts:
- U5: footprint Package_TO_SOT_SMD:SOT-666 -> Package_TO_SOT_SMD:SOT-23-6; LCSC C15999 -> C7519
Changed lines of the file:
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@@
       (effects (font (size 1.27 1.27)))
     )
-    (property "Footprint" "Package_TO_SOT_SMD:SOT-666" (at 115.57 194.31 0)
+    (property "Footprint" "Package_TO_SOT_SMD:SOT-23-6" (at 115.57 194.31 0)
       (effects (font (size 1.27 1.27)) hide)
     )
@@
       (effects (font (size 1.27 1.27)) hide)
     )
-    (property "LCSC" "C15999" (at 134.62 204.47 0)
+    (property "LCSC" "C7519" (at 134.62 204.47 0)
       (effects (font (size 1.27 1.27)) hide)
     )

Commit message: updates
Parts:
- J1: value Conn_01x04 -> Conn_01x05; footprint Connector_PinHeader_1.27mm:PinHeader_1x04_P1.27mm_Vertical -> Connector_PinHeader_1.27mm:PinHeader_1x05_P1.27mm_Vertical; symbol Connector_Generic:Conn_01x04 -> Connector_Generic:Conn_01x05
Connections:
- net COL0: now also U3.50 (PA15); no longer U3.46 (PA13)
- net COL1: now also U3.46 (PA13); no longer U3.50 (PA15)
- net COL10: now also U3.27 (PB1); no longer U3.34 (PB13)
- net COL2: now also U3.41 (PA8); no longer U3.27 (PB1)
- net COL3: now also U3.40 (PC9); no longer U3.41 (PA8)
- net COL4: now also U3.39 (PC8); no longer U3.40 (PC9)
- net COL5: now also U3.38 (PC7); no longer U3.39 (PC8)
- net COL6: now also U3.37 (PC6); no longer U3.38 (PC7)
- net COL7: now also U3.36 (PB15); no longer U3.37 (PC6)
- net COL8: now also U3.35 (PB14); no longer U3.36 (PB15)
- net COL9: now also U3.34 (PB13); no longer U3.35 (PB14)
- net PA9: now reaches U3.42 (PA9)
- net PA9: now also J1.5 (Pin_5)
- no-connect marks 4 -> 3
Changed lines of the file:
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@@
   )
   (no_connect (at 58.42 118.745))
-  (no_connect (at 162.56 104.14))
   (no_connect (at 181.61 106.68))
   (no_connect (at 53.34 106.045))
@@
     (effects (font (size 1.0922 1.0922)) (justify left bottom))
   )
-  (text "a9 forbidden\n" (at 163.83 105.41 0)
+  (text "a9 forbidden\n" (at 172.72 104.14 0)
     (effects (font (size 1.27 1.27)) (justify left bottom))
   )
@@
     )
   )
-  (global_label "COL10" (shape bidirectional) (at 182.88 154.94 0)
+  (global_label "COL10" (shape bidirectional) (at 162.56 127 0)
     (effects (font (size 1.27 1.27)) (justify left))
-    (property "Intersheetrefs" "${INTERSHEET_REFS}" (at 182.88 154.94 0)
+    (property "Intersheetrefs" "${INTERSHEET_REFS}" (at 162.56 127 0)
       (effects (font (size 1.27 1.27)) hide)
     )
@@
     )
   )
-  (global_label "COL3" (shape bidirectional) (at 162.56 101.6 0)
-    (effects (font (size 1.27 1.27)) (justify left))
-    (property "Intersheetrefs" "${INTERSHEET_REFS}" (at 162.56 101.6 0)
+  (global_label "COL3" (shape bidirectional) (at 124.46 144.78 180)
+    (effects (font (size 1.27 1.27)) (justify right))
+    (property "Intersheetrefs" "${INTERSHEET_REFS}" (at 124.46 144.78 0)
       (effects (font (size 1.27 1.27)) hide)
     )
@@
     )
   )
-  (global_label "COL5" (shape bidirectional) (at 124.46 142.24 180)
+  (global_label "COL5" (shape bidirectional) (at 124.46 139.7 180)
     (effects (font (size 1.27 1.27)) (justify right))
-    (property "Intersheetrefs" "${INTERSHEET_REFS}" (at 124.46 142.24 0)
+    (property "Intersheetrefs" "${INTERSHEET_REFS}" (at 124.46 139.7 0)
       (effects (font (size 1.27 1.27)) hide)
     )
@@
     )
   )
-  (global_label "COL1" (shape bidirectional) (at 162.56 119.38 0)
+  (global_label "COL1" (shape bidirectional) (at 162.56 114.3 0)
     (effects (font (size 1.27 1.27)) (justify left))
-    (property "Intersheetrefs" "${INTERSHEET_REFS}" (at 162.56 119.38 0)
+    (property "Intersheetrefs" "${INTERSHEET_REFS}" (at 162.56 114.3 0)
       (effects (font (size 1.27 1.27)) hide)
     )
@@
     )
   )
-  (global_label "COL9" (shape bidirectional) (at 162.56 157.48 0)
+  (global_label "COL9" (shape bidirectional) (at 182.88 154.94 0)
     (effects (font (size 1.27 1.27)) (justify left))
-    (property "Intersheetrefs" "${INTERSHEET_REFS}" (at 162.56 157.48 0)
+    (property "Intersheetrefs" "${INTERSHEET_REFS}" (at 182.88 154.94 0)
       (effects (font (size 1.27 1.27)) hide)
     )
@@
     )
   )
-  (global_label "PB6" (shape bidirectional) (at 54.61 218.44 0)
+  (global_label "PB6" (shape bidirectional) (at 54.61 220.98 0)
     (effects (font (size 1.27 1.27)) (justify left))
-    (property "Intersheetrefs" "${INTERSHEET_REFS}" (at 54.61 218.44 0)
+    (property "Intersheetrefs" "${INTERSHEET_REFS}" (at 54.61 220.98 0)
       (effects (font (size 1.27 1.27)) hide)
     )
@@
     )
   )
-  (global_label "COL4" (shape bidirectional) (at 124.46 144.78 180)
+  (global_label "COL4" (shape bidirectional) (at 124.46 142.24 180)
     (effects (font (size 1.27 1.27)) (justify right))
-    (property "Intersheetrefs" "${INTERSHEET_REFS}" (at 124.46 144.78 0)
+    (property "Intersheetrefs" "${INTERSHEET_REFS}" (at 124.46 142.24 0)
       (effects (font (size 1.27 1.27)) hide)
     )
@@
     )
   )
-  (global_label "COL7" (shape bidirectional) (at 124.46 137.16 180)
-    (effects (font (size 1.27 1.27)) (justify right))
-    (property "Intersheetrefs" "${INTERSHEET_REFS}" (at 124.46 137.16 0)
+  (global_label "COL7" (shape bidirectional) (at 162.56 160.02 0)
+    (effects (font (size 1.27 1.27)) (justify left))
+    (property "Intersheetrefs" "${INTERSHEET_REFS}" (at 162.56 160.02 0)
       (effects (font (size 1.27 1.27)) hide)
     )
@@
     )
   )
-  (global_label "COL8" (shape bidirectional) (at 162.56 160.02 0)
+  (global_label "COL8" (shape bidirectional) (at 162.56 157.48 0)
     (effects (font (size 1.27 1.27)) (justify left))
-    (property "Intersheetrefs" "${INTERSHEET_REFS}" (at 162.56 160.02 0)
+    (property "Intersheetrefs" "${INTERSHEET_REFS}" (at 162.56 157.48 0)
       (effects (font (size 1.27 1.27)) hide)
     )
@@
     )
   )
-  (global_label "PD2" (shape bidirectional) (at 54.61 220.98 0)
+  (global_label "PD2" (shape bidirectional) (at 54.61 223.52 0)
     (effects (font (size 1.27 1.27)) (justify left))
-    (property "Intersheetrefs" "${INTERSHEET_REFS}" (at 54.61 220.98 0)
+    (property "Intersheetrefs" "${INTERSHEET_REFS}" (at 54.61 223.52 0)
       (effects (font (size 1.27 1.27)) hide)
     )
@@
     )
   )
-  (global_label "COL6" (shape bidirectional) (at 124.46 139.7 180)
+  (global_label "COL6" (shape bidirectional) (at 124.46 137.16 180)
     (effects (font (size 1.27 1.27)) (justify right))
-    (property "Intersheetrefs" "${INTERSHEET_REFS}" (at 124.46 139.7 0)
+    (property "Intersheetrefs" "${INTERSHEET_REFS}" (at 124.46 137.16 0)
       (effects (font (size 1.27 1.27)) hide)
     )
@@
     )
   )
-  (global_label "PA10" (shape bidirectional) (at 54.61 215.9 0)
+  (global_label "PA10" (shape bidirectional) (at 54.61 218.44 0)
     (effects (font (size 1.27 1.27)) (justify left))
-    (property "Intersheetrefs" "${INTERSHEET_REFS}" (at 54.61 215.9 0)
+    (property "Intersheetrefs" "${INTERSHEET_REFS}" (at 54.61 218.44 0)
       (effects (font (size 1.27 1.27)) hide)
     )
@@
     )
   )
-  (global_label "PC12" (shape bidirectional) (at 54.61 223.52 0)
+  (global_label "PC12" (shape bidirectional) (at 54.61 226.06 0)
     (effects (font (size 1.27 1.27)) (justify left))
-    (property "Intersheetrefs" "${INTERSHEET_REFS}" (at 54.61 223.52 0)
+    (property "Intersheetrefs" "${INTERSHEET_REFS}" (at 54.61 226.06 0)
       (effects (font (size 1.27 1.27)) hide)
     )
@@
     )
   )
-  (global_label "COL2" (shape bidirectional) (at 162.56 127 0)
+  (global_label "COL2" (shape bidirectional) (at 162.56 101.6 0)
     (effects (font (size 1.27 1.27)) (justify left))
-    (property "Intersheetrefs" "${INTERSHEET_REFS}" (at 162.56 127 0)
+    (property "Intersheetrefs" "${INTERSHEET_REFS}" (at 162.56 101.6 0)
       (effects (font (size 1.27 1.27)) hide)
     )
@@
     )
   )
+  (global_label "PA9" (shape bidirectional) (at 54.61 215.9 0)
+    (effects (font (size 1.27 1.27)) (justify left))
+    (property "Intersheetrefs" "${INTERSHEET_REFS}" (at 54.61 215.9 0)
+      (effects (font (size 1.27 1.27)) hide)
+    )
+  )
   (global_label "ROW0" (shape bidirectional) (at 162.56 124.46 0)
     (effects (font (size 1.27 1.27)) (justify left))
@@
     )
   )
-  (global_label "COL0" (shape bidirectional) (at 162.56 114.3 0)
+  (global_label "COL0" (shape bidirectional) (at 162.56 119.38 0)
     (effects (font (size 1.27 1.27)) (justify left))
-    (property "Intersheetrefs" "${INTERSHEET_REFS}" (at 162.56 114.3 0)
+    (property "Intersheetrefs" "${INTERSHEET_REFS}" (at 162.56 119.38 0)
       (effects (font (size 1.27 1.27)) hide)
     )
@@
     )
   )
+  (global_label "PA9" (shape bidirectional) (at 162.56 104.14 0)
+    (effects (font (size 1.27 1.27)) (justify left))
+    (property "Intersheetrefs" "${INTERSHEET_REFS}" (at 162.56 104.14 0)
+      (effects (font (size 1.27 1.27)) hide)
+    )
+  )
   (symbol (lib_id "ws2812b:WS2812B") (at 274.32 135.89 0) (unit 1)
     (in_bom yes) (on_board yes) (dnp no)
@@
     )
   )
-  (symbol (lib_id "Connector_Generic:Conn_01x04") (at 49.53 220.98 180) (unit 1)
+  (symbol (lib_id "Connector_Generic:Conn_01x05") (at 49.53 220.98 180) (unit 1)
     (in_bom yes) (on_board yes) (dnp no) (fields_autoplaced)
     (property "Reference" "J1" (at 49.53 211.6201 0)
       (effects (font (size 1.27 1.27)))
     )
-    (property "Value" "Conn_01x04" (at 49.53 213.5411 0)
+    (property "Value" "Conn_01x05" (at 49.53 213.5411 0)
       (effects (font (size 1.27 1.27)))
     )
-    (property "Footprint" "Connector_PinHeader_1.27mm:PinHeader_1x04_P1.27mm_Vertical" (at 49.53 220.98 0)
+    (property "Footprint" "Connector_PinHeader_1.27mm:PinHeader_1x05_P1.27mm_Vertical" (at 49.53 220.98 0)
       (effects (font (size 1.27 1.27)) hide)
     )
@@
     (pin "3")
     (pin "4")
+    (pin "5")
     (instances
       (project "m0116"
