File: m0116.kicad_sch (KiCad schematic)
At the start: 262 parts, among them J1 Conn_01x05, J2 Conn_01x04_MountingPin, J3 Conn_01x04_MountingPin, J4 Conn_01x04, J7 Conn_01x05, Q1 Q_PMOS_GSD AO3401A, Q2 Q_NMOS_GSD 2N7002, Q3 Q_NMOS_GSD 2N7002, Q4 2N3904, SW1 SW_Push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

Commit message: fix
Parts:
- SW1: footprint random-keyboard-parts:SKQG-1155865 -> controller:switch_K2-1187SQ-A4SW-06
Changed lines of the file:
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@@
   (junction (at 160.02 314.96) (diameter 0) (color 0 0 0 0)
   )
-  (junction (at 36.83 35.56) (diameter 0) (color 0 0 0 0)
-  )
   (junction (at 143.51 361.95) (diameter 0) (color 0 0 0 0)
   )
@@
   (junction (at 167.64 323.85) (diameter 0) (color 0 0 0 0)
   )
+  (junction (at 36.83 36.83) (diameter 0) (color 0 0 0 0)
+  )
   (junction (at 86.36 386.08) (diameter 0) (color 0 0 0 0)
   )
@@
     (stroke (width 0) (type default))
   )
+  (wire (pts (xy 36.83 34.29) (xy 36.83 36.83))
+    (stroke (width 0) (type default))
+  )
   (wire (pts (xy 40.64 266.7) (xy 40.64 285.75))
     (stroke (width 0) (type solid))
@@
     (stroke (width 0) (type default))
   )
-  (wire (pts (xy 36.83 35.56) (xy 36.83 34.29))
-    (stroke (width 0) (type default))
-  )
   (wire (pts (xy 78.74 104.14) (xy 88.9 104.14))
     (stroke (width 0) (type default))
@@
     (stroke (width 0) (type solid))
   )
-  (wire (pts (xy 48.26 35.56) (xy 36.83 35.56))
+  (wire (pts (xy 49.53 36.83) (xy 36.83 36.83))
     (stroke (width 0) (type default))
   )
@@
     (stroke (width 0) (type default))
   )
-  (wire (pts (xy 36.83 38.1) (xy 36.83 35.56))
+  (wire (pts (xy 36.83 41.91) (xy 36.83 36.83))
     (stroke (width 0) (type default))
   )
@@
     )
   )
-  (symbol (lib_id "controller-rescue:GND-power") (at 36.83 38.1 0) (unit 1)
+  (symbol (lib_id "controller-rescue:GND-power") (at 36.83 41.91 0) (unit 1)
     (in_bom yes) (on_board yes) (dnp no)
-    (property "Reference" "#PWR023" (at 36.83 44.45 0)
+    (property "Reference" "#PWR023" (at 36.83 48.26 0)
       (effects (font (size 1.27 1.27)) hide)
     )
-    (property "Value" "GND" (at 36.957 42.4942 0)
+    (property "Value" "GND" (at 36.957 46.3042 0)
       (effects (font (size 1.27 1.27)))
     )
-    (property "Footprint" "" (at 36.83 38.1 0)
+    (property "Footprint" "" (at 36.83 41.91 0)
       (effects (font (size 1.27 1.27)) hide)
     )
-    (property "Datasheet" "" (at 36.83 38.1 0)
+    (property "Datasheet" "" (at 36.83 41.91 0)
       (effects (font (size 1.27 1.27)) hide)
     )
@@
       (effects (font (size 1.27 1.27)) (justify left))
     )
-    (property "Footprint" "random-keyboard-parts:SKQG-1155865" (at 63.5 112.395 0)
+    (property "Footprint" "controller:switch_K2-1187SQ-A4SW-06" (at 63.5 112.395 0)
       (effects (font (size 1.27 1.27)) hide)
     )
@@
     )
   )
-  (symbol (lib_id "controller-rescue:PWR_FLAG-power") (at 48.26 35.56 0) (unit 1)
+  (symbol (lib_id "controller-rescue:PWR_FLAG-power") (at 49.53 36.83 0) (unit 1)
     (in_bom yes) (on_board yes) (dnp no)
-    (property "Reference" "#FLG0103" (at 48.26 33.655 0)
+    (property "Reference" "#FLG0103" (at 49.53 34.925 0)
       (effects (font (size 1.27 1.27)) hide)
     )
-    (property "Value" "PWR_FLAG" (at 48.26 31.1658 0)
+    (property "Value" "PWR_FLAG" (at 49.53 32.4358 0)
       (effects (font (size 1.27 1.27)))
     )
-    (property "Footprint" "" (at 48.26 35.56 0)
+    (property "Footprint" "" (at 49.53 36.83 0)
       (effects (font (size 1.27 1.27)) hide)
     )
-    (property "Datasheet" "~" (at 48.26 35.56 0)
+    (property "Datasheet" "~" (at 49.53 36.83 0)
       (effects (font (size 1.27 1.27)) hide)
     )

Commit message: updates
Connections:
- net COL12: now also U3.58 (PB6); no longer U3.57 (PB5)
- net ROW3: now also U3.24 (PC4); no longer U3.25 (PC5)
- net PB6 renamed PB5
- net PB5: now also U3.57 (PB5); no longer U3.58 (PB6)
- net PC4 renamed PC5
- net PC5: now also U3.25 (PC5); no longer U3.24 (PC4)
Other:
- note added: "Note: PB5 and PC5 can be used for I2C, e.g., for OLED"
Changed lines of the file:
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@@
-(kicad_sch (version 20221206) (generator eeschema)
+(kicad_sch (version 20230221) (generator eeschema)
   (paper "C")
   (junction (at 217.17 304.8) (diameter 0) (color 0 0 0 0)
@@
     (effects (font (size 1.27 1.27)) (justify left bottom))
   )
+  (text "Note: PB5 and PC5 can be used for I2C, e.g., for OLED"
+    (at 22.86 234.95 0)
+    (effects (font (size 1.27 1.27)) (justify left bottom))
+  )
   (text "6.25u at101w\nfor quasi aek 2" (at 133.35 379.73 0)
     (effects (font (size 1.27 1.27)) (justify left bottom))
@@
     )
   )
-  (global_label "PC4" (shape bidirectional) (at 45.72 196.85 0)
+  (global_label "PC5" (shape bidirectional) (at 45.72 196.85 0)
     (effects (font (size 1.27 1.27)) (justify left))
     (property "Intersheetrefs" "${INTERSHEET_REFS}" (at 45.72 196.85 0)
@@
     )
   )
-  (global_label "PC4" (shape bidirectional) (at 124.46 132.08 180)
+  (global_label "PC5" (shape bidirectional) (at 124.46 134.62 180)
     (effects (font (size 1.27 1.27)) (justify right))
-    (property "Intersheetrefs" "${INTERSHEET_REFS}" (at 124.46 132.08 0)
+    (property "Intersheetrefs" "${INTERSHEET_REFS}" (at 124.46 134.62 0)
       (effects (font (size 1.27 1.27)) hide)
     )
@@
     )
   )
-  (global_label "PB6" (shape bidirectional) (at 54.61 220.98 0)
+  (global_label "PB5" (shape bidirectional) (at 54.61 220.98 0)
     (effects (font (size 1.27 1.27)) (justify left))
     (property "Intersheetrefs" "${INTERSHEET_REFS}" (at 54.61 220.98 0)
@@
     )
   )
-  (global_label "COL12" (shape bidirectional) (at 162.56 137.16 0)
+  (global_label "COL12" (shape bidirectional) (at 162.56 139.7 0)
     (effects (font (size 1.27 1.27)) (justify left))
-    (property "Intersheetrefs" "${INTERSHEET_REFS}" (at 162.56 137.16 0)
+    (property "Intersheetrefs" "${INTERSHEET_REFS}" (at 162.56 139.7 0)
       (effects (font (size 1.27 1.27)) hide)
     )
@@
     )
   )
-  (global_label "ROW3" (shape bidirectional) (at 124.46 134.62 180)
+  (global_label "ROW3" (shape bidirectional) (at 124.46 132.08 180)
     (effects (font (size 1.27 1.27)) (justify right))
-    (property "Intersheetrefs" "${INTERSHEET_REFS}" (at 124.46 134.62 0)
+    (property "Intersheetrefs" "${INTERSHEET_REFS}" (at 124.46 132.08 0)
       (effects (font (size 1.27 1.27)) hide)
     )
@@
     )
   )
-  (global_label "PB6" (shape bidirectional) (at 162.56 139.7 0)
+  (global_label "PB5" (shape bidirectional) (at 162.56 137.16 0)
     (effects (font (size 1.27 1.27)) (justify left))
-    (property "Intersheetrefs" "${INTERSHEET_REFS}" (at 162.56 139.7 0)
+    (property "Intersheetrefs" "${INTERSHEET_REFS}" (at 162.56 137.16 0)
       (effects (font (size 1.27 1.27)) hide)
     )
@@
       (effects (font (size 1.27 1.27)) hide)
     )
-    (property "Value" "+3.3V" (at 214.0712 79.121 90)
+    (property "Value" "+3V3" (at 214.0712 79.121 90)
       (effects (font (size 1.27 1.27)) (justify left))
     )
@@
       (effects (font (size 1.27 1.27)) hide)
     )
-    (property "Value" "+3.3V" (at 214.0712 89.281 90)
+    (property "Value" "+3V3" (at 214.0712 89.281 90)
       (effects (font (size 1.27 1.27)) (justify left))
     )
@@
       (effects (font (size 1.27 1.27)) hide)
     )
-    (property "Value" "+3.3V" (at 49.911 147.8788 90)
+    (property "Value" "+3V3" (at 49.911 147.8788 90)
       (effects (font (size 1.27 1.27)) (justify left))
     )
@@
       (effects (font (size 1.27 1.27)) hide)
     )
-    (property "Value" "+3.3V" (at 59.69 102.235 0)
+    (property "Value" "+3V3" (at 59.69 102.235 0)
       (effects (font (size 1.27 1.27)))
     )
@@
       (effects (font (size 1.27 1.27)) hide)
     )
-    (property "Value" "+3.3V" (at 241.681 15.9258 0)
+    (property "Value" "+3V3" (at 241.681 15.9258 0)
       (effects (font (size 1.27 1.27)))
     )
@@
       (effects (font (size 1.27 1.27)) hide)
     )
-    (property "Value" "+3.3V" (at 214.0712 84.201 90)
+    (property "Value" "+3V3" (at 214.0712 84.201 90)
       (effects (font (size 1.27 1.27)) (justify left))
     )
@@
       (effects (font (size 1.27 1.27)) hide)
     )
-    (property "Value" "+3.3V" (at 137.541 63.5508 0)
+    (property "Value" "+3V3" (at 137.541 63.5508 0)
       (effects (font (size 1.27 1.27)))
     )
@@
       (effects (font (size 1.27 1.27)) hide)
     )
-    (property "Value" "+3.3V" (at 204.851 45.1358 0)
+    (property "Value" "+3V3" (at 204.851 45.1358 0)
       (effects (font (size 1.27 1.27)))
     )
@@
       (effects (font (size 1.27 1.27)) hide)
     )
-    (property "Value" "+3.3V" (at 62.611 63.5508 0)
+    (property "Value" "+3V3" (at 62.611 63.5508 0)
       (effects (font (size 1.27 1.27)))
     )
@@
       (effects (font (size 1.27 1.27)) hide)
     )
-    (property "Value" "+3.3V" (at 79.121 18.4658 0)
+    (property "Value" "+3V3" (at 79.121 18.4658 0)
       (effects (font (size 1.27 1.27)))
     )
@@
       (effects (font (size 1.27 1.27)) hide)
     )
-    (property "Value" "+3.3V" (at 74.041 64.1858 0)
+    (property "Value" "+3V3" (at 74.041 64.1858 0)
       (effects (font (size 1.27 1.27)))
     )
@@
       (effects (font (size 1.27 1.27)) hide)
     )
-    (property "Value" "+3.3V" (at 173.101 24.8158 0)
+    (property "Value" "+3V3" (at 173.101 24.8158 0)
       (effects (font (size 1.27 1.27)))
     )

Commit message: updates
Parts:
- J1: value Conn_01x05 -> Conn_01x06; footprint Connector_PinHeader_1.27mm:PinHeader_1x05_P1.27mm_Vertical -> Connector_PinHeader_1.27mm:PinHeader_1x06_P1.27mm_Vertical; symbol Connector_Generic:Conn_01x05 -> Connector_Generic:Conn_01x06
Connections:
- net PA10: now also J1.5 (Pin_5); no longer J1.4 (Pin_4)
- net PA9: now also J1.6 (Pin_6); no longer J1.5 (Pin_5)
- net PB5: now also J1.4 (Pin_4); no longer J1.3 (Pin_3)
- net PC10: now also J1.1 (Pin_1)
- net PC12: now also J1.2 (Pin_2); no longer J1.1 (Pin_1)
- net PD2: now also J1.3 (Pin_3); no longer J1.2 (Pin_2)
Changed lines of the file:
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@@
     (effects (font (size 1.27 1.27)) (justify left bottom))
   )
+  (text "Note: PB5 and PC5 can be used for I2C, e.g., for OLED"
+    (at 22.86 237.49 0)
+    (effects (font (size 1.27 1.27)) (justify left bottom))
+  )
   (text "One per VDD pin" (at 181.61 27.305 0)
     (effects (font (size 1.27 1.27)) (justify left bottom))
@@
     )
   )
-  (global_label "PB5" (shape bidirectional) (at 54.61 220.98 0)
+  (global_label "PB5" (shape bidirectional) (at 59.69 218.44 0)
     (effects (font (size 1.27 1.27)) (justify left))
-    (property "Intersheetrefs" "${INTERSHEET_REFS}" (at 54.61 220.98 0)
+    (property "Intersheetrefs" "${INTERSHEET_REFS}" (at 59.69 218.44 0)
       (effects (font (size 1.27 1.27)) hide)
     )
@@
     )
   )
-  (global_label "PD2" (shape bidirectional) (at 54.61 223.52 0)
+  (global_label "PD2" (shape bidirectional) (at 59.69 220.98 0)
     (effects (font (size 1.27 1.27)) (justify left))
-    (property "Intersheetrefs" "${INTERSHEET_REFS}" (at 54.61 223.52 0)
+    (property "Intersheetrefs" "${INTERSHEET_REFS}" (at 59.69 220.98 0)
       (effects (font (size 1.27 1.27)) hide)
     )
@@
     )
   )
-  (global_label "PA10" (shape bidirectional) (at 54.61 218.44 0)
+  (global_label "PA10" (shape bidirectional) (at 59.69 215.9 0)
     (effects (font (size 1.27 1.27)) (justify left))
-    (property "Intersheetrefs" "${INTERSHEET_REFS}" (at 54.61 218.44 0)
+    (property "Intersheetrefs" "${INTERSHEET_REFS}" (at 59.69 215.9 0)
       (effects (font (size 1.27 1.27)) hide)
     )
@@
     )
   )
-  (global_label "PC12" (shape bidirectional) (at 54.61 226.06 0)
+  (global_label "PC12" (shape bidirectional) (at 59.69 223.52 0)
     (effects (font (size 1.27 1.27)) (justify left))
-    (property "Intersheetrefs" "${INTERSHEET_REFS}" (at 54.61 226.06 0)
+    (property "Intersheetrefs" "${INTERSHEET_REFS}" (at 59.69 223.52 0)
       (effects (font (size 1.27 1.27)) hide)
     )
@@
     )
   )
-  (global_label "PA9" (shape bidirectional) (at 54.61 215.9 0)
+  (global_label "PA9" (shape bidirectional) (at 59.69 213.36 0)
     (effects (font (size 1.27 1.27)) (justify left))
-    (property "Intersheetrefs" "${INTERSHEET_REFS}" (at 54.61 215.9 0)
+    (property "Intersheetrefs" "${INTERSHEET_REFS}" (at 59.69 213.36 0)
       (effects (font (size 1.27 1.27)) hide)
     )
@@
     )
   )
+  (global_label "PC10" (shape bidirectional) (at 59.69 226.06 0)
+    (effects (font (size 1.27 1.27)) (justify left))
+    (property "Intersheetrefs" "${INTERSHEET_REFS}" (at 59.69 226.06 0)
+      (effects (font (size 1.27 1.27)) hide)
+    )
+  )
   (global_label "COL7" (shape input) (at 151.13 259.08 90) (fields_autoplaced)
     (effects (font (size 1.27 1.27)) (justify left))
@@
     )
   )
-  (symbol (lib_id "Connector_Generic:Conn_01x05") (at 49.53 220.98 180) (unit 1)
+  (symbol (lib_id "Connector_Generic:Conn_01x06") (at 54.61 220.98 180) (unit 1)
     (in_bom yes) (on_board yes) (dnp no) (fields_autoplaced)
-    (property "Reference" "J1" (at 49.53 211.6201 0)
+    (property "Reference" "J1" (at 54.61 211.6201 0)
       (effects (font (size 1.27 1.27)))
     )
-    (property "Value" "Conn_01x05" (at 49.53 213.5411 0)
+    (property "Value" "Conn_01x06" (at 54.61 213.5411 0)
       (effects (font (size 1.27 1.27)))
     )
-    (property "Footprint" "Connector_PinHeader_1.27mm:PinHeader_1x05_P1.27mm_Vertical" (at 49.53 220.98 0)
+    (property "Footprint" "Connector_PinHeader_1.27mm:PinHeader_1x06_P1.27mm_Vertical" (at 54.61 220.98 0)
       (effects (font (size 1.27 1.27)) hide)
     )
-    (property "Datasheet" "~" (at 49.53 220.98 0)
+    (property "Datasheet" "~" (at 54.61 220.98 0)
       (effects (font (size 1.27 1.27)) hide)
     )
@@
     (pin "4")
     (pin "5")
+    (pin "6")
     (instances
       (project "m0116"
